Commit message: Improve arm demo motion stability and visuals

File: src/complete_description/urdf/Complete.xacro (robot description, xacro)
@@ -149,4 +149,5 @@
   <child link="link_2_1"/>
   <axis xyz="0.0 -1.0 0.0"/>
+  <dynamics damping="1.5" friction="0.25"/>
 </joint>
 <joint name="revolute_6" type="continuous">
@@ -155,4 +156,5 @@
   <child link="link_3_1"/>
   <axis xyz="0.0 1.0 -0.0"/>
+  <dynamics damping="1.5" friction="0.25"/>
 </joint>
 <joint name="revolute_7" type="continuous">
@@ -161,4 +163,5 @@
   <child link="link_4_1"/>
   <axis xyz="-0.0 1.0 -0.0"/>
+  <dynamics damping="1.2" friction="0.2"/>
 </joint>
 <joint name="revolute_8" type="continuous">
@@ -167,4 +170,5 @@
   <child link="link_5_1"/>
   <axis xyz="-1.0 -0.0 0.0"/>
+  <dynamics damping="1.0" friction="0.15"/>
 </joint>
 <joint name="revolute_12" type="continuous">
@@ -173,4 +177,5 @@
   <child link="link_6_1"/>
   <axis xyz="0.0 0.0 1.0"/>
+  <dynamics damping="0.8" friction="0.1"/>
 </joint>
 <joint name="revolute_13" type="continuous">
@@ -179,4 +184,5 @@
   <child link="link_1_1"/>
   <axis xyz="0.0 0.0 -1.0"/>
+  <dynamics damping="1.2" friction="0.2"/>
 </joint>
 </robot>
